Commit message: depth deprojections almost there. Restructured urdf/obj directories. Maybe for the worse.

File: src/pybullet_tree_sim/pybullet_tree_sim/urdf/trees/envy/macro/tree_macro.urdf.xacro (robot description, xacro)
@@ -13,5 +13,5 @@
             <visual>
                 <geometry>
-                    <mesh filename="./meshes/trees/envy/test/tree_${tree_id}.obj" scale="${scale}"/>
+                    <mesh filename="./meshes/trees/envy/unlabeled/obj/${namespace}${tree_type}_tree${tree_id}.obj" scale="${scale}"/>
                 </geometry>
                 <material name="LightGrey">
@@ -21,5 +21,5 @@
             <collision concave="true">
                 <geometry>
-                    <mesh filename="./meshes/trees/envy/test/tree_${tree_id}.obj" scale="${scale}"/>
+                    <mesh filename="./meshes/trees/envy/unlabeled/obj/${namespace}${tree_type}_tree${tree_id}.obj" scale="${scale}"/>
                 </geometry>
             </collision>
