Commit message: updates to robot description

File: src/branch_detection_system_description/urdf/end_effectors/mock_pruner/macro/mock_pruner_macro.urdf.xacro (robot description, xacro)
@@ -10,5 +10,5 @@
         <!-- static properties -->
         <xacro:property name="mock_pruner_mass" value="2.0" />
-        <xacro:property name="base__tool0_offset" value="0.0 0.0 0.27208"/>
+        <xacro:property name="base__tool0_offset" value="0.0 0.0 0.23508"/>
         <!-- <xacro:property name="base__tool0_offset" value="0.0 0.0 0.20"/> -->
         <xacro:property name="base__tof0_offset" value="${tof0_offset}"/>
@@ -16,5 +16,5 @@
         <!-- <xacro:property name="base__tof0_offset" value="${tof0_offset} 0 0.15"/> -->
         <!-- <xacro:property name="base__tof1_offset" value="${tof1_offset} 0 0.15"/> -->
-        <xacro:property name="base__camera0_offset" value="0.0 0.0600 0.19094"/>
+        <xacro:property name="base__camera0_offset" value="0.0 -0.069 0.16379"/>
         <!-- additional args -->
         <xacro:arg name="dovetail_male_mount_prefix" default="dovetail_male_mount__" />

Commit message: added solidworks files for custom eef

File: src/branch_detection_system_description/urdf/end_effectors/mock_pruner/macro/mock_pruner_macro.urdf.xacro (robot description, xacro)
@@ -10,5 +10,5 @@
         <!-- static properties -->
         <xacro:property name="mock_pruner_mass" value="0.256" />
-        <xacro:property name="base__tool0_offset" value="0.0 0.0 0.23508"/>
+        <xacro:property name="base__tool0_offset" value="0.0 0.0 0.15208"/>
         <!-- <xacro:property name="base__tool0_offset" value="0.0 0.0 0.20"/> -->
         <xacro:property name="base__tof0_offset" value="${tof0_offset}"/>

File: src/branch_detection_system_description/urdf/tmp/robot.urdf (robot description, URDF)
Before this commit: robot pruning_robot, 30 links, 29 joints
Joints:
- joint mock_pruner__base--tof0: origin xyz=0.1 -0.015 0.21737 rpy=0 0 0 -> xyz=0.04891 -0.02373 0.14237 rpy=0 0 0
- joint mock_pruner__base--tof1: origin xyz=-0.1 -0.015 0.21737 rpy=0 0 0 -> xyz=-0.04891 -0.02373 0.14237 rpy=0 0 0
- joint mock_pruner__base--tool0: origin xyz=0.0 0.0 0.23508 rpy=0 0 0 -> xyz=0.0 0.0 0.15208 rpy=0 0 0
