Commit message: added rotational offset link, updated measured masses

File: src/branch_detection_system_description/urdf/end_effectors/dovetail_mount/macro/dovetail_mount_macro.urdf.xacro (robot description, xacro)
@@ -4,4 +4,5 @@
     <xacro:property name="dovetail_female_tool0_height" value="0.023"/>
     <xacro:property name="dovetail_male_rot_offset" value="0.0 0.0 0.0"/>
+    <xacro:property name="dovetail_remale_rot_offset" value="0.0 0.0 0.0"/>
     <xacro:macro name="dovetail_male_mount_macro" params="parent_link dovetail_male_mount_prefix mesh_base_path">
         <!-- ==================== -->
@@ -11,5 +12,5 @@
             <color rgba="0.749 0.580 0.894 1"/>
         </material>
-        <xacro:property name="dovetail_male_mass" value="0.025"/>
+        <xacro:property name="dovetail_male_mass" value="0.033"/>
         <!-- links -->
         <link name="${dovetail_male_mount_prefix}base"/>
@@ -59,5 +60,5 @@
             <color rgba="0.929 0.710 0.145 1"/>
         </material>
-        <xacro:property name="dovetail_female_mass" value="0.025"/>
+        <xacro:property name="dovetail_female_mass" value="0.038"/>
         <!-- links -->
         <link name="${dovetail_female_mount_prefix}base"/>

File: src/branch_detection_system_description/urdf/end_effectors/mock_pruner/macro/mock_pruner_macro.urdf.xacro (robot description, xacro)
@@ -7,7 +7,7 @@
     <xacro:property name="mock_pruner_rot_offset" value="0.0 0.0 0.0"/>
     <!-- Materials -->
-    <xacro:macro name="mock_pruner_macro" params="parent_link eef_prefix tof0_offset tof1_offset camera_offset mesh_base_path urdf_base_path">
+    <xacro:macro name="mock_pruner_macro" params="parent_link eef_prefix tof0_offset tof1_offset camera_offset mesh_base_path">
         <!-- static properties -->
-        <xacro:property name="mock_pruner_mass" value="2.0" />
+        <xacro:property name="mock_pruner_mass" value="0.256" />
         <xacro:property name="base__tool0_offset" value="0.0 0.0 0.23508"/>
         <!-- <xacro:property name="base__tool0_offset" value="0.0 0.0 0.20"/> -->
@@ -18,12 +18,19 @@
         <xacro:property name="base__camera0_offset" value="0.0 -0.069 0.16379"/>
         <!-- additional args -->
+        <xacro:arg name="rotation_correction_plate_prefix" default="rotation_correction_plate__" />
         <xacro:arg name="dovetail_male_mount_prefix" default="dovetail_male_mount__" />
         <xacro:arg name="dovetail_female_mount_prefix" default="dovetail_female_mount__" />
         <xacro:arg name="mesh_base_path" default=""/>
-        <xacro:arg name="urdf_base_path" default=""/>
+        <!-- rotation correction plate macro -->
+        <xacro:include filename="$(find branch_detection_system_description)/urdf/end_effectors/rotation_correction_plate/macro/rotation_correction_plate_macro.urdf.xacro" />
+        <xacro:rotation_correction_plate_macro
+            parent_link="${parent_link}"
+            rotation_correction_plate_prefix="$(arg rotation_correction_plate_prefix)"
+            mesh_base_path="${mesh_base_path}"
+        />
         <!-- dovetail_mount macro -->
-        <xacro:include filename="${urdf_base_path}/end_effectors/dovetail_mount/macro/dovetail_mount_macro.urdf.xacro" />
+        <xacro:include filename="$(find branch_detection_system_description)/urdf/end_effectors/dovetail_mount/macro/dovetail_mount_macro.urdf.xacro" />
         <xacro:dovetail_mount_macro
-            parent_link="${parent_link}"
+            parent_link="$(arg rotation_correction_plate_prefix)tool0"
             dovetail_male_mount_prefix="$(arg dovetail_male_mount_prefix)"
             dovetail_female_mount_prefix="$(arg dovetail_female_mount_prefix)"

File: src/branch_detection_system_description/urdf/robot/robot.urdf.xacro (robot description, xacro)
@@ -7,5 +7,4 @@
     <xacro:arg name="robot_stack_qty" default='0'/>
     <xacro:arg name="mesh_base_path" default=''/>
-    <xacro:arg name="urdf_base_path" default=''/>
     <!-- generate generic robot with stack_qty number of links, link parents -->
     <xacro:macro name='arg_assignment_loop' params='stack_qty'>
@@ -116,5 +115,5 @@
             <!-- Robot cart -->
             <xacro:if value="${ str(resolved_part) == 'cart' }">
-                <xacro:include filename="$(arg urdf_base_path)/base_mounts/cart/macro/cart_macro.urdf.xacro"/>
+                <xacro:include filename="$(find branch_detection_system_description)/urdf/base_mounts/cart/macro/cart_macro.urdf.xacro"/>
                 <xacro:cart_macro
                     cart_prefix="cart__"
@@ -124,5 +123,5 @@
             </xacro:if>
             <xacro:if value="${ str(resolved_part) == 'mock_pruner' }">
-                <xacro:include filename="$(arg urdf_base_path)/end_effectors/mock_pruner/macro/mock_pruner_macro.urdf.xacro"/>
+                <xacro:include filename="$(find branch_detection_system_description)/urdf/end_effectors/mock_pruner/macro/mock_pruner_macro.urdf.xacro"/>
                 <!-- Args -->
                 <xacro:arg name="mock_pruner_prefix" default="mock_pruner__" />
@@ -135,5 +134,4 @@
                     parent_link="${resolved_parent_link}"
                     mesh_base_path="$(arg mesh_base_path)"
-                    urdf_base_path="$(arg urdf_base_path)"
                     tof0_offset='$(arg tof0_offset)'
                     tof1_offset='$(arg tof1_offset)'

Commit message: updated URDF to include rotational offset piece

File: src/branch_detection_system_description/urdf/end_effectors/dovetail_mount/macro/dovetail_mount_macro.urdf.xacro (robot description, xacro)
@@ -1,8 +1,4 @@
 <?xml version="1.0"?>
 <robot xmlns:xacro="https://ros.org/wiki/xacro" name="dovetail_mount">
-    <xacro:property name="dovetail_male_tool0_height" value="0.008"/>
-    <xacro:property name="dovetail_female_tool0_height" value="0.023"/>
-    <xacro:property name="dovetail_male_rot_offset" value="0.0 0.0 0.0"/>
-    <xacro:property name="dovetail_remale_rot_offset" value="0.0 0.0 0.0"/>
     <xacro:macro name="dovetail_male_mount_macro" params="parent_link dovetail_male_mount_prefix mesh_base_path">
         <!-- ==================== -->
@@ -13,4 +9,6 @@
         </material>
         <xacro:property name="dovetail_male_mass" value="0.033"/>
+        <xacro:property name="dovetail_male_tool0_height" value="0.008"/>
+        <xacro:property name="dovetail_male_rot_offset" value="0.0 0.0 0.0"/>
         <!-- links -->
         <link name="${dovetail_male_mount_prefix}base"/>
@@ -61,4 +59,6 @@
         </material>
         <xacro:property name="dovetail_female_mass" value="0.038"/>
+        <xacro:property name="dovetail_female_tool0_height" value="0.023"/>
+        <xacro:property name="dovetail_female_rot_offset" value="0.0 0.0 ${pi}"/>
         <!-- links -->
         <link name="${dovetail_female_mount_prefix}base"/>
@@ -86,5 +86,5 @@
         <!-- joints -->
         <joint name="${parent_link}--${dovetail_female_mount_prefix}base" type="fixed">
-            <origin xyz="0 0 ${dovetail_female_tool0_height}" rpy="0 0 0"/>
+            <origin xyz="0 0 ${dovetail_female_tool0_height}" rpy="${dovetail_female_rot_offset}"/>
             <parent link="${parent_link}"/>
             <child link="${dovetail_female_mount_prefix}base"/>

File: src/branch_detection_system_description/urdf/end_effectors/mock_pruner/macro/mock_pruner_macro.urdf.xacro (robot description, xacro)
@@ -5,5 +5,5 @@
     <!-- <xacro:arg name="mesh_base_path" default="./"/> -->
     <!-- <xacro:property name="end_effector_parent" value="" /> -->
-    <xacro:property name="mock_pruner_rot_offset" value="0.0 0.0 0.0"/>
+    <xacro:property name="mock_pruner_rot_offset" value="0.0 0.0 ${pi}"/>
     <!-- Materials -->
     <xacro:macro name="mock_pruner_macro" params="parent_link eef_prefix tof0_offset tof1_offset camera_offset mesh_base_path">
@@ -76,5 +76,5 @@
         <!-- ================== -->
         <joint name="$(arg dovetail_female_mount_prefix)tool0--${eef_prefix}base" type="fixed">
-            <origin xyz="0 0 0" rpy="0 0 0"/>
+            <origin xyz="0 0 0" rpy="${mock_pruner_rot_offset}"/>
             <parent link="$(arg dovetail_female_mount_prefix)tool0"/>
             <child link="${eef_prefix}base"/>

File: src/branch_detection_system_description/urdf/end_effectors/rotation_correction_plate/macro/rotation_correction_plate_macro.urdf.xacro (robot description, xacro)
@@ -4,4 +4,5 @@
     <xacro:property name="rotation_correction_plate_rot_offset" value="0.0 0.0 0.0"/>
     <xacro:property name="rotation_correction_plate_mass" value="0.047"/>
+    <xacro:property name="rotation_correction_plate_rot_offset" value="0.0 0.0 ${pi}" />
     <xacro:macro name="rotation_correction_plate_macro" params="parent_link rotation_correction_plate_prefix mesh_base_path">
         <!-- =========================== -->

File: src/branch_detection_system_moveit_config/srdf/robot_macro.srdf.xacro (robot description, xacro)
@@ -55,5 +55,13 @@
     <disable_collisions link1="${prefix}wrist_2_link" link2="${prefix}wrist_3_link" reason="Adjacent" />
     <!-- TODO Dynamically configure. Can probably be done with just the "body" links? Or maybe virtual links here. -->
-    <disable_collisions link1="dovetail_male_mount__base" link2="${prefix}tool0" reason="Adjacent" />
+    <disable_collisions link1="rotation_correction_plate__base" link2="${prefix}tool0" reason="Adjacent" />
+    <disable_collisions link1="rotation_correction_plate__base" link2="${prefix}wrist_3_link" reason="Never" />
+    <disable_collisions link1="rotation_correction_plate__body" link2="${prefix}tool0" reason="Adjacent" />
+    <disable_collisions link1="rotation_correction_plate__body" link2="${prefix}wrist_3_link" reason="Never" />
+    <disable_collisions link1="rotation_correction_plate__body" link2="dovetail_male_mount__base" reason="Adjacent" />
+    <disable_collisions link1="rotation_correction_plate__body" link2="dovetail_male_mount__body" reason="Never" />
+    <disable_collisions link1="rotation_correction_plate__tool0" link2="dovetail_male_mount__base" reason="Adjacent" />
+    <disable_collisions link1="rotation_correction_plate__tool0" link2="dovetail_male_mount__body" reason="Never" />
+    <disable_collisions link1="dovetail_male_mount__base" link2="${prefix}tool0" reason="Never" />
     <disable_collisions link1="dovetail_male_mount__base" link2="dovetail_male_mount__body" reason="Never" />
     <disable_collisions link1="dovetail_male_mount__base" link2="dovetail_male_mount__tool0" reason="Never" />

Commit message: updates to description urdf/stl files

File: src/branch_detection_system_description/urdf/end_effectors/dovetail_mount/macro/dovetail_mount_macro.urdf.xacro (robot description, xacro)
@@ -9,5 +9,5 @@
         </material>
         <xacro:property name="dovetail_male_mass" value="0.033"/>
-        <xacro:property name="dovetail_male_tool0_height" value="0.008"/>
+        <xacro:property name="dovetail_male_tool0_height" value="0.02293"/>
         <xacro:property name="dovetail_male_rot_offset" value="0.0 0.0 0.0"/>
         <!-- links -->
@@ -59,6 +59,6 @@
         </material>
         <xacro:property name="dovetail_female_mass" value="0.038"/>
-        <xacro:property name="dovetail_female_tool0_height" value="0.023"/>
-        <xacro:property name="dovetail_female_rot_offset" value="0.0 0.0 ${pi}"/>
+        <xacro:property name="dovetail_female_tool0_height" value="0.008"/>
+        <xacro:property name="dovetail_female_rot_offset" value="0.0 0.0 0.0"/>
         <!-- links -->
         <link name="${dovetail_female_mount_prefix}base"/>
@@ -86,5 +86,5 @@
         <!-- joints -->
         <joint name="${parent_link}--${dovetail_female_mount_prefix}base" type="fixed">
-            <origin xyz="0 0 ${dovetail_female_tool0_height}" rpy="${dovetail_female_rot_offset}"/>
+            <origin xyz="0 0 0.0" rpy="${dovetail_female_rot_offset}"/>
             <parent link="${parent_link}"/>
             <child link="${dovetail_female_mount_prefix}base"/>
@@ -96,5 +96,5 @@
         </joint>
         <joint name="${dovetail_female_mount_prefix}body--tool0" type="fixed">
-            <origin xyz="0 0 0" rpy="0 0 0"/>
+            <origin xyz="0 0 ${dovetail_female_tool0_height}" rpy="0 0 0"/>
             <parent link="${dovetail_female_mount_prefix}body"/>
             <child link="${dovetail_female_mount_prefix}tool0"/>

File: src/branch_detection_system_description/urdf/end_effectors/mock_pruner/macro/mock_pruner_macro.urdf.xacro (robot description, xacro)
@@ -5,10 +5,10 @@
     <!-- <xacro:arg name="mesh_base_path" default="./"/> -->
     <!-- <xacro:property name="end_effector_parent" value="" /> -->
-    <xacro:property name="mock_pruner_rot_offset" value="0.0 0.0 ${pi}"/>
+    <xacro:property name="mock_pruner_rot_offset" value="0.0 0.0 0.0"/>
     <!-- Materials -->
     <xacro:macro name="mock_pruner_macro" params="parent_link eef_prefix tof0_offset tof1_offset camera_offset mesh_base_path">
         <!-- static properties -->
         <xacro:property name="mock_pruner_mass" value="0.256" />
-        <xacro:property name="base__tool0_offset" value="0.0 0.0 0.15208"/>
+        <xacro:property name="base__tool0_offset" value="0.0 0.0050825 0.1601525"/>
         <!-- <xacro:property name="base__tool0_offset" value="0.0 0.0 0.20"/> -->
         <xacro:property name="base__tof0_offset" value="${tof0_offset}"/>
@@ -16,5 +16,5 @@
         <!-- <xacro:property name="base__tof0_offset" value="${tof0_offset} 0 0.15"/> -->
         <!-- <xacro:property name="base__tof1_offset" value="${tof1_offset} 0 0.15"/> -->
-        <xacro:property name="base__camera0_offset" value="0.0 -0.069 0.16379"/>
+        <xacro:property name="base__camera0_offset" value="-0.0017977 -0.0715747 0.0711646"/>
         <!-- additional args -->
         <xacro:arg name="rotation_correction_plate_prefix" default="rotation_correction_plate__" />

File: src/branch_detection_system_description/urdf/end_effectors/rotation_correction_plate/macro/rotation_correction_plate_macro.urdf.xacro (robot description, xacro)
@@ -4,5 +4,5 @@
     <xacro:property name="rotation_correction_plate_rot_offset" value="0.0 0.0 0.0"/>
     <xacro:property name="rotation_correction_plate_mass" value="0.047"/>
-    <xacro:property name="rotation_correction_plate_rot_offset" value="0.0 0.0 ${pi}" />
+    <xacro:property name="rotation_correction_plate_rot_offset" value="0.0 0.0 0.0" />
     <xacro:macro name="rotation_correction_plate_macro" params="parent_link rotation_correction_plate_prefix mesh_base_path">
         <!-- =========================== -->

File: src/branch_detection_system_description/urdf/tmp/robot.urdf (robot description, URDF)
Before this commit: robot pruning_robot, 30 links, 29 joints
Joints:
- joint dovetail_female_mount__body--tool0: origin xyz=0 0 0 rpy=0 0 0 -> xyz=0 0 0.008 rpy=0 0 0
- joint dovetail_female_mount__tool0--mock_pruner__base: origin xyz=0 0 0 rpy=0.0 0.0 3.141592653589793 -> xyz=0 0 0 rpy=0.0 0.0 0.0
- joint dovetail_male_mount__body--tool0: origin xyz=0 0 0.008 rpy=0 0 0 -> xyz=0 0 0.02293 rpy=0 0 0
- joint dovetail_male_mount__tool0--dovetail_female_mount__base: origin xyz=0 0 0.023 rpy=0.0 0.0 3.141592653589793 -> xyz=0 0 0.0 rpy=0.0 0.0 0.0
- joint mock_pruner__base--camera0: origin xyz=0.0 -0.069 0.16379 rpy=0 0 0 -> xyz=-0.0017977 -0.0715747 0.0711646 rpy=0 0 0
- joint mock_pruner__base--tof0: origin xyz=0.04891 -0.02373 0.14237 rpy=0 0 0 -> xyz=0.04891 0.005 0.14237 rpy=0 0 0
- joint mock_pruner__base--tof1: origin xyz=-0.04891 -0.02373 0.14237 rpy=0 0 0 -> xyz=-0.04891 0.005 0.14237 rpy=0 0 0
- joint mock_pruner__base--tool0: origin xyz=0.0 0.0 0.15208 rpy=0 0 0 -> xyz=0.0 0.0050825 0.1601525 rpy=0 0 0
- joint ur5e__tool0--rotation_correction_plate__base: origin xyz=0 0 0 rpy=0.0 0.0 3.141592653589793 -> xyz=0 0 0 rpy=0.0 0.0 0.0
