Commit message: adding dynamic urdf to description pkg

File: src/branch_detection_system_description/urdf/base_mounts/cart/macro/cart_macro.urdf.xacro (robot description, xacro)
@@ -20,5 +20,5 @@
             <origin rpy="0.0 0.0 0.0" xyz="0.0 0.0 ${cart_collision_box_z}"/>
             <geometry>
-                <mesh filename="${mesh_base_path}/base_mounts/cart/cart.obj"/>
+                <mesh filename="file://$(find branch_detection_system_description)/meshes/base_mounts/cart/cart.obj"/>
             </geometry>
             <material name="LightGrey"/>

File: src/branch_detection_system_description/urdf/end_effectors/dovetail_mount/macro/dovetail_mount_macro.urdf.xacro (robot description, xacro)
@@ -3,5 +3,5 @@
     <xacro:property name="dovetail_male_tool0_height" value="0.008"/>
     <xacro:property name="dovetail_female_tool0_height" value="0.023"/>
-    <xacro:property name="dovetail_male_rot_offset" value="0.0 0.0 ${pi}"/>
+    <xacro:property name="dovetail_male_rot_offset" value="0.0 0.0 0.0"/>
     <xacro:macro name="dovetail_male_mount_macro" params="parent_link dovetail_male_mount_prefix mesh_base_path">
         <!-- ==================== -->
@@ -19,5 +19,5 @@
                 <origin xyz="0 0 0" rpy="0 0 0"/>
                 <geometry>
-                    <mesh filename="${mesh_base_path}/end_effectors/dovetail/DovetailMale.STL"/>
+                    <mesh filename="file://$(find branch_detection_system_description)/meshes/end_effectors/dovetail/DovetailMale.STL"/>
                 </geometry>
             </visual>
@@ -25,5 +25,5 @@
                 <origin xyz="0 0 0" rpy="0 0 0"/>
                 <geometry>
-                    <mesh filename="${mesh_base_path}/end_effectors/dovetail/DovetailMale.STL"/>
+                    <mesh filename="file://$(find branch_detection_system_description)/meshes/end_effectors/dovetail/DovetailMale.STL"/>
                 </geometry>
             </collision>
@@ -67,5 +67,5 @@
                 <origin xyz="0 0 0" rpy="0 0 0"/>
                 <geometry>
-                    <mesh filename="${mesh_base_path}/end_effectors/dovetail/DovetailFemale.STL"/>
+                    <mesh filename="file://$(find branch_detection_system_description)/meshes/end_effectors/dovetail/DovetailFemale.STL"/>
                 </geometry>
             </visual>
@@ -73,5 +73,5 @@
                 <origin xyz="0 0 0" rpy="0 0 0"/>
                 <geometry>
-                    <mesh filename="${mesh_base_path}/end_effectors/dovetail/DovetailFemale.STL"/>
+                    <mesh filename="file://$(find branch_detection_system_description)/meshes/end_effectors/dovetail/DovetailFemale.STL"/>
                 </geometry>
             </collision>

File: src/branch_detection_system_description/urdf/end_effectors/mock_pruner/macro/mock_pruner_macro.urdf.xacro (robot description, xacro)
@@ -12,6 +12,6 @@
         <xacro:property name="base__tool0_offset" value="0.0 0.0 0.27208"/>
         <!-- <xacro:property name="base__tool0_offset" value="0.0 0.0 0.20"/> -->
-        <xacro:property name="base__tof0_offset" value="${tof0_offset} 0 0.142"/>
-        <xacro:property name="base__tof1_offset" value="${tof1_offset} 0 0.142"/>
+        <xacro:property name="base__tof0_offset" value="${tof0_offset}"/>
+        <xacro:property name="base__tof1_offset" value="${tof1_offset}"/>
         <!-- <xacro:property name="base__tof0_offset" value="${tof0_offset} 0 0.15"/> -->
         <!-- <xacro:property name="base__tof1_offset" value="${tof1_offset} 0 0.15"/> -->
@@ -43,5 +43,5 @@
                 <origin xyz="0 0 0" rpy="0 0 0"/>
                 <geometry>
-                    <mesh filename="${mesh_base_path}/end_effectors/mock_pruner/MockPruner.STL" />
+                    <mesh filename="file://$(find branch_detection_system_description)/meshes/end_effectors/mock_pruner/MockPruner.STL" />
                 </geometry>
             </visual>
@@ -49,5 +49,5 @@
                 <origin xyz="0 0 0" rpy="0 0 0"/>
                 <geometry>
-                    <mesh filename="${mesh_base_path}/end_effectors/mock_pruner/MockPruner.STL" />
+                    <mesh filename="file://$(find branch_detection_system_description)/meshes/end_effectors/mock_pruner/MockPruner.STL" />
                 </geometry>
             </collision>

Commit message: fixed default cart tool0 mount position

File: src/branch_detection_system_description/urdf/base_mounts/cart/macro/cart_macro.urdf.xacro (robot description, xacro)
@@ -12,4 +12,5 @@
     <xacro:property name="cart_collision_box_y" value='1.0'/>
     <xacro:property name="cart_collision_box_z" value='0.75711'/>
+    <xacro:property name="cart_tool0_mount_rotation" value="0.0 0.0 -${pi/4}"/>
     <!-- ================== -->
     <!--       Links        -->
@@ -57,5 +58,5 @@
     </joint>
     <joint name="${cart_prefix}cart--${cart_prefix}tool0" type="fixed">
-        <origin rpy="0 0 0" xyz="0 0 ${cart_collision_box_z}"/>
+        <origin rpy="${cart_tool0_mount_rotation}" xyz="0 0 ${cart_collision_box_z}"/>
         <parent link="${cart_prefix}cart"/>
         <child link="${cart_prefix}tool0"/>
