Commit message: made changes to add amiga base. still needs better configuration for switching bases, but should work for now

File: src/branch_detection_system_description/urdf/base_mounts/farm-ng/macro/amiga_macro.urdf.xacro (robot description, xacro)
@@ -9,9 +9,16 @@
     </material>
     <xacro:property name="amiga_mass" value="40.0"/>
-    <xacro:property name="amiga_collision_box_x" value='1.132'/>
-    <xacro:property name="amiga_collision_box_y" value='0.800'/>
-    <xacro:property name="amiga_collision_box_z" value='1.339'/>
-    <xacro:property name="amiga_tool0_mount_rotation" value="0.0 0.0 0.0"/>
-    <xacro:property name="amiga_tool0_mount_position" value="0.12825037 0.323256 0.99810607"/>
+    <xacro:property name="amiga_collision_box0_x" value='1.132'/>
+    <xacro:property name="amiga_collision_box0_y" value='0.800'/>
+    <xacro:property name="amiga_collision_box0_z" value='0.99810607'/>
+    <xacro:property name="amiga_collision_box1_x" value='${amiga_collision_box0_x}' />
+    <xacro:property name="amiga_collision_box1_y" value='0.6' />
+    <xacro:property name="amiga_collision_box1_z" value='0.2' />
+    <xacro:property name="amiga_collision_box2_x" value='0.25' />
+    <xacro:property name="amiga_collision_box2_y" value='0.25' />
+    <xacro:property name="amiga_collision_box2_z" value='0.25' />
+    <xacro:property name="amiga_tool0_mount_rotation" value="0.0 0.0 -${pi / 4}"/>
+    <!-- <xacro:property name="amiga_tool0_mount_position" value="-0.12825037 0.323256 0.99810607"/> -->
+    <xacro:property name="amiga_tool0_mount_position" value="-0.4 0.323256 0.99810607"/>
     <!-- ================== -->
     <!--       Links        -->
@@ -20,14 +27,26 @@
     <link name="${amiga_prefix}body">
         <visual>
-            <origin rpy="0.0 0.0 0.0" xyz="0.0 0.0 ${amiga_collision_box_z}"/>
+            <origin rpy="0.0 0.0 0.0" xyz="0.0 0.0 0.0"/>
             <geometry>
-                <mesh filename="file://$(find branch_detection_system_description)/meshes/base_mounts/farm-ng/amiga/frame_on_amiga_v2.STL"/>
+                <mesh filename="file://$(find branch_detection_system_description)/meshes/base_mounts/farm-ng/amiga/frame_on_amiga_v2_simplified.stl"/>
             </geometry>
             <material name="LightLightGrey"/>
         </visual>
         <collision>
-            <origin rpy="0.0 0.0 0.0" xyz="0.0 0.0 0.0"/>
+            <origin rpy="0.0 0.0 0.0" xyz="0.0 0.0 ${amiga_collision_box0_z / 2}"/>
             <geometry>
-                <box size="${amiga_collision_box_x} ${amiga_collision_box_y} ${amiga_collision_box_z}"/>
+                <box size="${amiga_collision_box0_x} ${amiga_collision_box0_y} ${amiga_collision_box0_z}"/>
+            </geometry>
+        </collision>
+        <collision>
+            <origin rpy="0.0 0.0 0.0" xyz="0.0 -${amiga_collision_box1_y / 5} ${amiga_collision_box0_z}" />
+            <geometry>
+                <box size="${amiga_collision_box1_x} ${amiga_collision_box1_y} ${amiga_collision_box1_z}" />
+            </geometry>
+        </collision>
+        <collision>
+            <origin rpy="0.0 0.0 0.0" xyz="${amiga_collision_box0_x / 2 - amiga_collision_box2_x / 2} ${amiga_collision_box2_y / 3} ${amiga_collision_box0_z + amiga_collision_box1_z}" />
+            <geometry>
+                <box size="${amiga_collision_box2_x} ${amiga_collision_box2_y} ${amiga_collision_box2_z}" />
             </geometry>
         </collision>
@@ -35,10 +54,10 @@
             <origin rpy="0 0 0" xyz="0.0 0.0 0.0"/>
             <mass value="${amiga_mass}"/>
-            <inertia ixx="${1/12 * amiga_mass * (amiga_collision_box_y**2 + amiga_collision_box_z**2)}"
+            <inertia ixx="${1/12 * amiga_mass * (amiga_collision_box0_y**2 + amiga_collision_box0_z**2)}"
                      ixz="0.0"
                      ixy="0.0"
-                     iyy="${1/12 * amiga_mass * (amiga_collision_box_x**2 + amiga_collision_box_z**2)}"
+                     iyy="${1/12 * amiga_mass * (amiga_collision_box0_x**2 + amiga_collision_box0_z**2)}"
                      iyz="0.0"
-                     izz="${1/12 * amiga_mass * (amiga_collision_box_y**2 + amiga_collision_box_x**2)}"
+                     izz="${1/12 * amiga_mass * (amiga_collision_box0_y**2 + amiga_collision_box0_x**2)}"
             />
         </inertial>

File: src/branch_detection_system_description/urdf/tmp/robot.urdf (robot description, URDF)
Before this commit: robot pruning_robot, 30 links, 29 joints
Links:
- removed link cart__base
- removed link cart__cart
- removed link cart__tool0
- added link amiga__base
- added link amiga__body, mass 40.0; collision box size=0.25 0.25 0.25; collision box size=1.132 0.6 0.2
- added link amiga__tool0
Joints:
- removed joint cart__base--cart__cart
- removed joint cart__cart--cart__tool0
- removed joint world--cart__base
- added joint amiga__base--amiga__body: type fixed, parent amiga__base, child amiga__body, origin xyz=0 0 0 rpy=0 0 0
- added joint amiga__body--amiga__tool0: type fixed, parent amiga__body, child amiga__tool0, origin xyz=-0.4 0.323256 0.99810607 rpy=0.0 0.0 -0.7853981633974483
- added joint world--amiga__base: type fixed, parent world, child amiga__base, origin xyz=0 0 0 rpy=0 0 0
- joint ur5e__base_joint: parent cart__tool0 -> amiga__tool0

File: src/branch_detection_system_moveit_config/srdf/robot.srdf.xacro (robot description, xacro)
@@ -5,5 +5,5 @@
   <!-- parameters -->
   <xacro:arg name="ur_prefix" default="ur5e__" />
-  <xacro:include filename="$(find branch_detection_system_moveit_config)/srdf/robot_macro.srdf.xacro"/>
+  <xacro:include filename="$(find branch_detection_system_moveit_config)/srdf/robot_amiga_macro.srdf.xacro"/>
   <xacro:ur_srdf name="$(arg name)" arm_prefix="$(arg ur_prefix)"/>
 </robot>

Commit message: minor edits for amiga workflow. ready to test

File: src/branch_detection_system_description/urdf/base_mounts/farm-ng/macro/amiga_macro.urdf.xacro (robot description, xacro)
@@ -18,7 +18,7 @@
     <xacro:property name="amiga_collision_box2_y" value='0.25' />
     <xacro:property name="amiga_collision_box2_z" value='0.25' />
-    <xacro:property name="amiga_tool0_mount_rotation" value="0.0 0.0 -${pi / 4}"/>
+    <xacro:property name="amiga_tool0_mount_rotation" value="0.0 0.0 -${pi / 4 + pi}"/>
     <!-- <xacro:property name="amiga_tool0_mount_position" value="-0.12825037 0.323256 0.99810607"/> -->
-    <xacro:property name="amiga_tool0_mount_position" value="-0.4 0.323256 0.99810607"/>
+    <xacro:property name="amiga_tool0_mount_position" value="-0.225 0.323256 0.99810607"/>
     <!-- ================== -->
     <!--       Links        -->
