Commit message: added in dynamic variable prefix-ing to yaml files

File: src/branch_detection_system_description/urdf/tmp/robot.urdf (robot description, URDF)
Before this commit: robot pruning_robot, 30 links, 29 joints
Joints:
- joint cart__cart--cart__tool0: origin xyz=0 0 0.75711 rpy=0 0 0 -> xyz=0 0 0.75711 rpy=0.0 0.0 -0.7853981633974483

File: src/branch_detection_system_moveit_config/srdf/robot.srdf.xacro (robot description, xacro)
@@ -4,6 +4,6 @@
   <xacro:arg name="name" default="ur"/>
   <!-- parameters -->
-  <xacro:arg name="prefix" default="ur5e__" />
+  <xacro:arg name="ur_prefix" default="ur5e__" />
   <xacro:include filename="$(find branch_detection_system_moveit_config)/srdf/robot_macro.srdf.xacro"/>
-  <xacro:ur_srdf name="$(arg name)" prefix="$(arg prefix)"/>
+  <xacro:ur_srdf name="$(arg name)" arm_prefix="$(arg ur_prefix)"/>
 </robot>

File: src/branch_detection_system_moveit_config/srdf/robot_macro.srdf.xacro (robot description, xacro)
@@ -5,5 +5,5 @@
     A URDF file must exist for this robot as well, where the joints and the links that are referenced are defined
 -->
-  <xacro:macro name="ur_srdf" params="name prefix">
+  <xacro:macro name="ur_srdf" params="name arm_prefix">
     <!--GROUPS - Representation of a set of joints and links. This can be useful for specifying DOF to plan for, defining arms, end effectors, etc-->
     <!--LINKS - When a link is specified, the parent joint of that link (if it exists) is automatically included-->
@@ -11,32 +11,32 @@
     <!--CHAINS - When a chain is specified, all the links along the chain (including endpoints) are included in the group. Additionally, all the joints that are parents to included links are also included. This means that joints along the chain and the parent joint of the base link are included in the group-->
     <!--SUBGROUPS - Groups can also be formed by referencing to already defined group names-->
-    <group name="${prefix}${name}_manipulator">
+    <group name="${arm_prefix}${name}_manipulator">
       <chain base_link="cart__base" tip_link="mock_pruner__tool0" />
-      <end_effector name="mock_pruner__eef" group="${prefix}${name}_manipulator" parent_link="mock_pruner__tool0"/>
+      <end_effector name="mock_pruner__eef" group="${arm_prefix}${name}_manipulator" parent_link="mock_pruner__tool0"/>
     </group>
     <!--GROUP STATES - Purpose - Define a named state for a particular group, in terms of joint values. This is useful to define states like 'folded arms'-->
-    <group_state name="${prefix}home" group="${prefix}${name}_manipulator">
-      <joint name="${prefix}elbow_joint" value="0" />
-      <joint name="${prefix}shoulder_lift_joint" value="-1.5707" />
-      <joint name="${prefix}shoulder_pan_joint" value="0" />
-      <joint name="${prefix}wrist_1_joint" value="0" />
-      <joint name="${prefix}wrist_2_joint" value="0" />
-      <joint name="${prefix}wrist_3_joint" value="0" />
+    <group_state name="${arm_prefix}home" group="${arm_prefix}${name}_manipulator">
+      <joint name="${arm_prefix}elbow_joint" value="0" />
+      <joint name="${arm_prefix}shoulder_lift_joint" value="-1.5707" />
+      <joint name="${arm_prefix}shoulder_pan_joint" value="0" />
+      <joint name="${arm_prefix}wrist_1_joint" value="0" />
+      <joint name="${arm_prefix}wrist_2_joint" value="0" />
+      <joint name="${arm_prefix}wrist_3_joint" value="0" />
     </group_state>
-    <group_state name="${prefix}up" group="${prefix}${name}_manipulator">
-      <joint name="${prefix}elbow_joint" value="0" />
-      <joint name="${prefix}shoulder_lift_joint" value="-1.5707" />
-      <joint name="${prefix}shoulder_pan_joint" value="0" />
-      <joint name="${prefix}wrist_1_joint" value="-1.5707" />
-      <joint name="${prefix}wrist_2_joint" value="0" />
-      <joint name="${prefix}wrist_3_joint" value="0" />
+    <group_state name="${arm_prefix}up" group="${arm_prefix}${name}_manipulator">
+      <joint name="${arm_prefix}elbow_joint" value="0" />
+      <joint name="${arm_prefix}shoulder_lift_joint" value="-1.5707" />
+      <joint name="${arm_prefix}shoulder_pan_joint" value="0" />
+      <joint name="${arm_prefix}wrist_1_joint" value="-1.5707" />
+      <joint name="${arm_prefix}wrist_2_joint" value="0" />
+      <joint name="${arm_prefix}wrist_3_joint" value="0" />
     </group_state>
-    <group_state name="${prefix}test_configuration" group="${prefix}${name}_manipulator">
-      <joint name="${prefix}elbow_joint" value="1.4" />
-      <joint name="${prefix}shoulder_lift_joint" value="-1.62" />
-      <joint name="${prefix}shoulder_pan_joint" value="1.54" />
-      <joint name="${prefix}wrist_1_joint" value="-1.2" />
-      <joint name="${prefix}wrist_2_joint" value="-1.6" />
-      <joint name="${prefix}wrist_3_joint" value="-0.11" />
+    <group_state name="${arm_prefix}test_configuration" group="${arm_prefix}${name}_manipulator">
+      <joint name="${arm_prefix}elbow_joint" value="1.4" />
+      <joint name="${arm_prefix}shoulder_lift_joint" value="-1.62" />
+      <joint name="${arm_prefix}shoulder_pan_joint" value="1.54" />
+      <joint name="${arm_prefix}wrist_1_joint" value="-1.2" />
+      <joint name="${arm_prefix}wrist_2_joint" value="-1.6" />
+      <joint name="${arm_prefix}wrist_3_joint" value="-0.11" />
     </group_state>
     <!--END EFFECTOR - Purpose - Represent information about an end effector.-->
@@ -47,35 +47,35 @@
     <disable_collisions link1="cart__tool0" link2="ur5e__base_link_inertia" reason="Never" />
     <disable_collisions link1="cart__tool0" link2="ur5e__base_link" reason="Never" />
-    <disable_collisions link1="${prefix}base_link" link2="${prefix}base_link_inertia" reason="Adjacent" />
-    <disable_collisions link1="${prefix}base_link_inertia" link2="${prefix}shoulder_link" reason="Adjacent" />
-    <disable_collisions link1="${prefix}tool0" link2="${prefix}wrist_1_link" reason="Never" />
-    <disable_collisions link1="${prefix}tool0" link2="${prefix}wrist_2_link" reason="Never" />
-    <disable_collisions link1="${prefix}tool0" link2="${prefix}wrist_3_link" reason="Adjacent" />
-    <disable_collisions link1="${prefix}forearm_link" link2="${prefix}upper_arm_link" reason="Adjacent" />
-    <disable_collisions link1="${prefix}forearm_link" link2="${prefix}wrist_1_link" reason="Adjacent" />
-    <disable_collisions link1="${prefix}shoulder_link" link2="${prefix}upper_arm_link" reason="Adjacent" />
-    <disable_collisions link1="${prefix}wrist_1_link" link2="${prefix}wrist_2_link" reason="Adjacent" />
-    <disable_collisions link1="${prefix}wrist_1_link" link2="${prefix}wrist_3_link" reason="Never" />
-    <disable_collisions link1="${prefix}wrist_2_link" link2="${prefix}wrist_3_link" reason="Adjacent" />
+    <disable_collisions link1="${arm_prefix}base_link" link2="${arm_prefix}base_link_inertia" reason="Adjacent" />
+    <disable_collisions link1="${arm_prefix}base_link_inertia" link2="${arm_prefix}shoulder_link" reason="Adjacent" />
+    <disable_collisions link1="${arm_prefix}tool0" link2="${arm_prefix}wrist_1_link" reason="Never" />
+    <disable_collisions link1="${arm_prefix}tool0" link2="${arm_prefix}wrist_2_link" reason="Never" />
+    <disable_collisions link1="${arm_prefix}tool0" link2="${arm_prefix}wrist_3_link" reason="Adjacent" />
+    <disable_collisions link1="${arm_prefix}forearm_link" link2="${arm_prefix}upper_arm_link" reason="Adjacent" />
+    <disable_collisions link1="${arm_prefix}forearm_link" link2="${arm_prefix}wrist_1_link" reason="Adjacent" />
+    <disable_collisions link1="${arm_prefix}shoulder_link" link2="${arm_prefix}upper_arm_link" reason="Adjacent" />
+    <disable_collisions link1="${arm_prefix}wrist_1_link" link2="${arm_prefix}wrist_2_link" reason="Adjacent" />
+    <disable_collisions link1="${arm_prefix}wrist_1_link" link2="${arm_prefix}wrist_3_link" reason="Never" />
+    <disable_collisions link1="${arm_prefix}wrist_2_link" link2="${arm_prefix}wrist_3_link" reason="Adjacent" />
     <!-- TODO Dynamically configure. Can probably be done with just the "body" links? Or maybe virtual links here. -->
-    <disable_collisions link1="rotation_correction_plate__base" link2="${prefix}tool0" reason="Adjacent" />
-    <disable_collisions link1="rotation_correction_plate__base" link2="${prefix}wrist_3_link" reason="Never" />
-    <disable_collisions link1="rotation_correction_plate__body" link2="${prefix}tool0" reason="Adjacent" />
-    <disable_collisions link1="rotation_correction_plate__body" link2="${prefix}wrist_3_link" reason="Never" />
+    <disable_collisions link1="rotation_correction_plate__base" link2="${arm_prefix}tool0" reason="Adjacent" />
+    <disable_collisions link1="rotation_correction_plate__base" link2="${arm_prefix}wrist_3_link" reason="Never" />
+    <disable_collisions link1="rotation_correction_plate__body" link2="${arm_prefix}tool0" reason="Adjacent" />
+    <disable_collisions link1="rotation_correction_plate__body" link2="${arm_prefix}wrist_3_link" reason="Never" />
     <disable_collisions link1="rotation_correction_plate__body" link2="dovetail_male_mount__base" reason="Adjacent" />
     <disable_collisions link1="rotation_correction_plate__body" link2="dovetail_male_mount__body" reason="Never" />
     <disable_collisions link1="rotation_correction_plate__tool0" link2="dovetail_male_mount__base" reason="Adjacent" />
     <disable_collisions link1="rotation_correction_plate__tool0" link2="dovetail_male_mount__body" reason="Never" />
-    <disable_collisions link1="dovetail_male_mount__base" link2="${prefix}tool0" reason="Never" />
+    <disable_collisions link1="dovetail_male_mount__base" link2="${arm_prefix}tool0" reason="Never" />
     <disable_collisions link1="dovetail_male_mount__base" link2="dovetail_male_mount__body" reason="Never" />
     <disable_collisions link1="dovetail_male_mount__base" link2="dovetail_male_mount__tool0" reason="Never" />
-    <disable_collisions link1="dovetail_male_mount__body" link2="${prefix}tool0" reason="Never"/>
-    <disable_collisions link1="dovetail_male_mount__body" link2="${prefix}wrist_3_link" reason="Never"/>
+    <disable_collisions link1="dovetail_male_mount__body" link2="${arm_prefix}tool0" reason="Never"/>
+    <disable_collisions link1="dovetail_male_mount__body" link2="${arm_prefix}wrist_3_link" reason="Never"/>
     <disable_collisions link1="dovetail_female_mount__base" link2="dovetail_male_mount__tool0" reason="Adjacent" />
     <disable_collisions link1="dovetail_female_mount__base" link2="dovetail_male_mount__body" reason="Adjacent" />
     <disable_collisions link1="dovetail_female_mount__body" link2="dovetail_male_mount__body" reason="Never" />
     <disable_collisions link1="dovetail_female_mount__body" link2="dovetail_male_mount__tool0" reason="Never" />
-    <disable_collisions link1="dovetail_female_mount__body" link2="${prefix}wrist_3_link" reason="Never"/>
-    <disable_collisions link1="dovetail_female_mount__body" link2="${prefix}tool0" reason="Never"/>
+    <disable_collisions link1="dovetail_female_mount__body" link2="${arm_prefix}wrist_3_link" reason="Never"/>
+    <disable_collisions link1="dovetail_female_mount__body" link2="${arm_prefix}tool0" reason="Never"/>
     <disable_collisions link1="mock_pruner__base" link2="dovetail_female_mount__tool0" reason="Adjacent" />
     <disable_collisions link1="mock_pruner__base" link2="dovetail_female_mount__body" reason="Never" />

Commit message: added pitch wrist controller files

File: src/branch_detection_system_description/urdf/tmp/robot.urdf (robot description, URDF)
Before this commit: robot pruning_robot, 30 links, 29 joints
Joints:
- joint amiga__body--amiga__tool0: origin xyz=-0.4 0.323256 0.99810607 rpy=0.0 0.0 -0.7853981633974483 -> xyz=-0.225 0.323256 0.99810607 rpy=0.0 0.0 -3.9269908169872414
