Commit message: field debug stuff

File: src/branch_detection_system/branch_detection_system_description/urdf/base_mounts/farm-ng/macro/amiga_macro.urdf.xacro (robot description, xacro)
@@ -18,5 +18,6 @@
     <xacro:property name="amiga_collision_box2_y" value='0.25' />
     <xacro:property name="amiga_collision_box2_z" value='0.25' />
-    <xacro:property name="amiga_tool0_mount_rotation" value="0.0 0.0 -${pi / 4 + pi}"/>
+    <!-- <xacro:property name="amiga_tool0_mount_rotation" value="0.0 0.0 -${pi / 4 + pi}"/> -->
+    <xacro:property name="amiga_tool0_mount_rotation" value="0.0 0.0 ${pi + pi/4}"/>
     <!-- <xacro:property name="amiga_tool0_mount_position" value="-0.12825037 0.323256 0.99810607"/> -->
     <xacro:property name="amiga_tool0_mount_position" value="-0.225 0.323256 0.99810607"/>

Commit message: got rough test BT working, fixed mount point in description

File: src/branch_detection_system/branch_detection_system_description/urdf/base_mounts/farm-ng/macro/amiga_macro.urdf.xacro (robot description, xacro)
@@ -20,5 +20,5 @@
     <xacro:property name="amiga_tool0_mount_rotation" value="0.0 0.0 -${pi / 4 + pi}"/>
     <!-- <xacro:property name="amiga_tool0_mount_position" value="-0.12825037 0.323256 0.99810607"/> -->
-    <xacro:property name="amiga_tool0_mount_position" value="-0.225 0.323256 0.99810607"/>
+    <xacro:property name="amiga_tool0_mount_position" value="-0.225 0.323256 ${0.99810607+0.1}"/>
     <!-- ================== -->
     <!--       Links        -->

Commit message: minor edits to rviz, xacro files

File: src/branch_detection_system/branch_detection_system_description/urdf/base_mounts/farm-ng/macro/amiga_macro.urdf.xacro (robot description, xacro)
@@ -18,5 +18,6 @@
     <xacro:property name="amiga_collision_box2_y" value='0.25' />
     <xacro:property name="amiga_collision_box2_z" value='0.25' />
-    <xacro:property name="amiga_tool0_mount_rotation" value="0.0 0.0 -${pi / 4 + pi}"/>
+    <!-- <xacro:property name="amiga_tool0_mount_rotation" value="0.0 0.0 -${pi / 4 + pi}"/> -->
+    <xacro:property name="amiga_tool0_mount_rotation" value="0.0 0.0 0.0"/>
     <!-- <xacro:property name="amiga_tool0_mount_position" value="-0.12825037 0.323256 0.99810607"/> -->
     <xacro:property name="amiga_tool0_mount_position" value="-0.225 0.323256 ${0.99810607+0.1}"/>
