Commit message: edits to the system description for new parts. Will likely make a new package for this in the future

File: branch_detection_system_description/urdf/base_mounts/farm-ng/macro/amiga_macro.urdf.xacro (robot description, xacro)
@@ -18,6 +18,6 @@
     <xacro:property name="amiga_collision_box2_y" value='0.25' />
     <xacro:property name="amiga_collision_box2_z" value='0.25' />
-    <!-- <xacro:property name="amiga_tool0_mount_rotation" value="0.0 0.0 -${pi / 4 + pi}"/> -->
-    <xacro:property name="amiga_tool0_mount_rotation" value="0.0 0.0 0.0"/>
+    <xacro:property name="amiga_tool0_mount_rotation" value="0.0 0.0 ${pi / 4}"/>
+    <!-- <xacro:property name="amiga_tool0_mount_rotation" value="0.0 0.0 0.0"/> -->
     <!-- <xacro:property name="amiga_tool0_mount_position" value="-0.12825037 0.323256 0.99810607"/> -->
     <xacro:property name="amiga_tool0_mount_position" value="-0.225 0.323256 ${0.99810607+0.1}"/>

File: branch_detection_system_description/urdf/end_effectors/mock_pruner/macro/mock_pruner_macro.urdf.xacro (robot description, xacro)
@@ -10,5 +10,5 @@
         <!-- static properties -->
         <xacro:property name="mock_pruner_mass" value="0.256" />
-        <xacro:property name="base__tool0_offset" value="0.0 0.0050825 0.1601525"/>
+        <xacro:property name="base__tool0_offset" value="0.0 0.0 0.1601525"/>
         <!-- <xacro:property name="base__tool0_offset" value="0.0 0.0 0.20"/> -->
         <xacro:property name="base__tof0_offset" value="${tof0_offset}"/>

File: branch_detection_system_description/urdf/robot/robot.urdf.xacro (robot description, xacro)
@@ -12,4 +12,5 @@
             <xacro:arg name="parent${stack_qty - 1}" default="world"/>
             <xacro:arg name="robot_part${stack_qty - 1}" default="world"/>
+            <!-- Recursively call macro -->
             <xacro:arg_assignment_loop stack_qty="${stack_qty - 1}"/>
         </xacro:if>

File: branch_detection_system_description/urdf/tmp/robot.urdf (robot description, URDF)
Before this commit: robot pruning_robot, 30 links, 29 joints
Joints:
- joint amiga__body--amiga__tool0: origin xyz=-0.225 0.323256 0.99810607 rpy=0.0 0.0 -3.9269908169872414 -> xyz=-0.225 0.323256 1.09810607 rpy=0.0 0.0 0.7853981633974483
